Commit message: added controllers for the robot arm

File: robot_arm_description/urdf/robot_arm.xacro (robot description, xacro)
@@ -1,4 +1,5 @@
 <?xml version="1.0" ?>
 <robot name="robot_arm" xmlns:xacro="http://www.ros.org/wiki/xacro">
+  <link name="world"/>
   <link name="base_link">
     <inertial>
@@ -177,4 +178,9 @@
     </collision>
   </link>
+  <joint name="world2base_joint" type="fixed">
+    <parent link="world"/>
+    <child link="base_link"/>
+    <dynamics damping="10" friction="1.0"/>
+  </joint>
   <joint name="shoulder_joint" type="revolute">
     <origin xyz="0.03435 0.0 0.194998" rpy="0 0 0"/>
@@ -275,3 +281,71 @@
     <selfCollide>true</selfCollide>
   </gazebo>
+  <!-- Ros2 Control Interface  -->
+  <gazebo>
+    <plugin filename="libgazebo_ros2_control.so" name="gazebo_ros2_control">
+      <robot_sim_type>gazebo_ros2_control/GazeboSystem</robot_sim_type>
+      <parameters>$(find robot_arm_description)/config/controller.yaml</parameters>
+    </plugin>
+  </gazebo>
+  <ros2_control name="GazeboSystem" type="system">
+    <hardware>
+      <plugin>gazebo_ros2_control/GazeboSystem</plugin>
+    </hardware>
+    <joint name="shoulder_joint">
+      <command_interface name="position">
+        <param name="min">-3.14</param>
+        <param name="max">3.14</param>
+      </command_interface>
+      <state_interface name="position"/>
+      <param name="initial_position">0.0</param>
+    </joint>
+    <joint name="elbow_joint">
+      <command_interface name="position">
+        <param name="min">-3.14</param>
+        <param name="max">3.14</param>
+      </command_interface>
+      <state_interface name="position"/>
+      <param name="initial_position">-1.57</param>
+    </joint>
+    <joint name="wrist_joint">
+      <command_interface name="position">
+        <param name="min">-3.14</param>
+        <param name="max">3.14</param>
+      </command_interface>
+      <state_interface name="position"/>
+      <param name="initial_position">0.0</param>
+    </joint>
+    <joint name="gripper_lower_joint">
+      <command_interface name="position">
+        <param name="min">-3.14</param>
+        <param name="max">3.14</param>
+      </command_interface>
+      <state_interface name="position"/>
+      <param name="initial_position">0.0</param>
+    </joint>
+    <joint name="gripper_joint">
+      <command_interface name="position">
+        <param name="min">-3.14</param>
+        <param name="max">3.14</param>
+      </command_interface>
+      <state_interface name="position"/>
+      <param name="initial_position">0.0</param>
+    </joint>
+    <joint name="finger1_joint">
+      <command_interface name="position">
+        <param name="min">-3.14</param>
+        <param name="max">3.14</param>
+      </command_interface>
+      <state_interface name="position"/>
+      <param name="initial_position">0.0</param>
+    </joint>
+    <joint name="finger2_joint">
+      <command_interface name="position">
+        <param name="min">-3.14</param>
+        <param name="max">3.14</param>
+      </command_interface>
+      <state_interface name="position"/>
+      <param name="initial_position">0.0</param>
+    </joint>
+  </ros2_control>
 </robot>

Commit message: added base_link to world joint

File: robot_arm_description/urdf/robot_arm.xacro (robot description, xacro)
@@ -4,4 +4,6 @@
 <xacro:include filename="$(find robot_arm_description)/urdf/robot_arm.trans" />
 <xacro:include filename="$(find robot_arm_description)/urdf/robot_arm.gazebo" />
+<link name="world">
+</link>
 <link name="base_link">
   <inertial>
@@ -504,4 +506,10 @@
   </collision>
 </link>
+<joint name="base_link_joint" type="fixed">
+  <origin xyz="0.0 0.0 0.0" rpy="0 0 0"/>
+  <parent link="world"/>
+  <child link="base_link"/>
+  <axis xyz="0.0 0.0 0.0"/>
+</joint>
 <joint name="pulley1_joint" type="fixed">
   <origin xyz="0.0 -0.00049 0.12851" rpy="0 0 0"/>

Commit message: added ros2_control controllers

File: robot_arm_description/urdf/robot_arm.xacro (robot description, xacro)
@@ -4,4 +4,6 @@
 <xacro:include filename="$(find robot_arm_description)/urdf/robot_arm.trans" />
 <xacro:include filename="$(find robot_arm_description)/urdf/robot_arm.gazebo" />
+<link name="world">
+</link>
 <link name="base_link">
   <inertial>
@@ -177,10 +179,10 @@
     <material name="opaque1965339"/>
   </visual>
-  <collision>
+  <!-- <collision>
     <origin xyz="0.0 -0.071 -0.166028" rpy="0 0 0"/>
     <geometry>
       <mesh filename="file://$(find robot_arm_description)/meshes/motor1_1.stl" scale="0.001 0.001 0.001"/>
     </geometry>
-  </collision>
+  </collision> -->
 </link>
 <link name="pulley2_1">
@@ -217,10 +219,10 @@
     <material name="opaque202209238"/>
   </visual>
-  <collision>
+  <!-- <collision>
     <origin xyz="0.097184 5e-05 -0.211028" rpy="0 0 0"/>
     <geometry>
       <mesh filename="file://$(find robot_arm_description)/meshes/motor2_1.stl" scale="0.001 0.001 0.001"/>
     </geometry>
-  </collision>
+  </collision> -->
 </link>
 <link name="pulley3_1">
@@ -317,10 +319,10 @@
     <material name="opaque1965339"/>
   </visual>
-  <collision>
+  <!-- <collision>
     <origin xyz="0.064839 -4.1e-05 -0.453571" rpy="0 0 0"/>
     <geometry>
       <mesh filename="file://$(find robot_arm_description)/meshes/motor3_1.stl" scale="0.001 0.001 0.001"/>
     </geometry>
-  </collision>
+  </collision> -->
 </link>
 <link name="motor4_1">
@@ -337,10 +339,10 @@
     <material name="opaque1965339"/>
   </visual>
-  <collision>
+  <!-- <collision>
     <origin xyz="-0.009222 -0.048743 -0.682474" rpy="0 0 0"/>
     <geometry>
       <mesh filename="file://$(find robot_arm_description)/meshes/motor4_1.stl" scale="0.001 0.001 0.001"/>
     </geometry>
-  </collision>
+  </collision> -->
 </link>
 <link name="pulley5_1">
@@ -424,5 +426,5 @@
   </collision>
 </link>
-<link name="motor5_1">
+<!-- <link name="motor5_1">
   <inertial>
     <origin xyz="0.05605440241182951 2.6991544145205104e-05 -2.1876837808743055e-05" rpy="0 0 0"/>
@@ -443,5 +445,5 @@
     </geometry>
   </collision>
-</link>
+</link> -->
 <link name="motor6_1">
   <inertial>
@@ -457,10 +459,10 @@
     <material name="steel_satin"/>
   </visual>
-  <collision>
+  <!-- <collision>
     <origin xyz="0.065393 0.259656 -0.629224" rpy="0 0 0"/>
     <geometry>
       <mesh filename="file://$(find robot_arm_description)/meshes/motor6_1.stl" scale="0.001 0.001 0.001"/>
     </geometry>
-  </collision>
+  </collision> -->
 </link>
 <link name="camera_mount_1">
@@ -504,4 +506,10 @@
   </collision>
 </link>
+<joint name="base_link_joint" type="fixed">
+  <origin xyz="0.0 0.0 0.0" rpy="0 0 0"/>
+  <parent link="world"/>
+  <child link="base_link"/>
+  <axis xyz="0.0 0.0 0.0"/>
+</joint>
 <joint name="pulley1_joint" type="fixed">
   <origin xyz="0.0 -0.00049 0.12851" rpy="0 0 0"/>
@@ -614,9 +622,9 @@
   <child link="pulley8_1"/>
 </joint>
-<joint name="motor5_joint" type="fixed">
+<!-- <joint name="motor5_joint" type="fixed">
   <origin xyz="-0.060986 -0.036531 0.0005" rpy="0 0 0"/>
   <parent link="table4_1"/>
   <child link="motor5_1"/>
-</joint>
+</joint> -->
 <joint name="motor6_joint" type="fixed">
   <origin xyz="-0.066956 -0.086535 0.0005" rpy="0 0 0"/>

Commit message: added ros2_control and controllers

File: robot_arm_description/urdf/robot_arm.xacro (robot description, xacro)
@@ -4,4 +4,6 @@
 <xacro:include filename="$(find robot_arm_description)/urdf/robot_arm.trans" />
 <xacro:include filename="$(find robot_arm_description)/urdf/robot_arm.gazebo" />
+<xacro:arg name="sim_gazebo" default="false" />
+<xacro:arg name="sim_gz" default="false" />
 <link name="world">
 </link>
@@ -179,10 +181,10 @@
     <material name="opaque1965339"/>
   </visual>
-  <collision>
+  <!-- <collision>
     <origin xyz="0.0 -0.071 -0.166028" rpy="0 0 0"/>
     <geometry>
       <mesh filename="file://$(find robot_arm_description)/meshes/motor1_1.stl" scale="0.001 0.001 0.001"/>
     </geometry>
-  </collision>
+  </collision> -->
 </link>
 <link name="pulley2_1">
@@ -219,10 +221,10 @@
     <material name="opaque202209238"/>
   </visual>
-  <collision>
+  <!-- <collision>
     <origin xyz="0.097184 5e-05 -0.211028" rpy="0 0 0"/>
     <geometry>
       <mesh filename="file://$(find robot_arm_description)/meshes/motor2_1.stl" scale="0.001 0.001 0.001"/>
     </geometry>
-  </collision>
+  </collision> -->
 </link>
 <link name="pulley3_1">
@@ -319,10 +321,10 @@
     <material name="opaque1965339"/>
   </visual>
-  <collision>
+  <!-- <collision>
     <origin xyz="0.064839 -4.1e-05 -0.453571" rpy="0 0 0"/>
     <geometry>
       <mesh filename="file://$(find robot_arm_description)/meshes/motor3_1.stl" scale="0.001 0.001 0.001"/>
     </geometry>
-  </collision>
+  </collision> -->
 </link>
 <link name="motor4_1">
@@ -339,10 +341,10 @@
     <material name="opaque1965339"/>
   </visual>
-  <collision>
+  <!-- <collision>
     <origin xyz="-0.009222 -0.048743 -0.682474" rpy="0 0 0"/>
     <geometry>
       <mesh filename="file://$(find robot_arm_description)/meshes/motor4_1.stl" scale="0.001 0.001 0.001"/>
     </geometry>
-  </collision>
+  </collision> -->
 </link>
 <link name="pulley5_1">
@@ -426,5 +428,5 @@
   </collision>
 </link>
-<link name="motor5_1">
+<!-- <link name="motor5_1">
   <inertial>
     <origin xyz="0.05605440241182951 2.6991544145205104e-05 -2.1876837808743055e-05" rpy="0 0 0"/>
@@ -445,5 +447,5 @@
     </geometry>
   </collision>
-</link>
+</link> -->
 <link name="motor6_1">
   <inertial>
@@ -459,10 +461,10 @@
     <material name="steel_satin"/>
   </visual>
-  <collision>
+  <!-- <collision>
     <origin xyz="0.065393 0.259656 -0.629224" rpy="0 0 0"/>
     <geometry>
       <mesh filename="file://$(find robot_arm_description)/meshes/motor6_1.stl" scale="0.001 0.001 0.001"/>
     </geometry>
-  </collision>
+  </collision> -->
 </link>
 <link name="camera_mount_1">
@@ -622,9 +624,9 @@
   <child link="pulley8_1"/>
 </joint>
-<joint name="motor5_joint" type="fixed">
+<!-- <joint name="motor5_joint" type="fixed">
   <origin xyz="-0.060986 -0.036531 0.0005" rpy="0 0 0"/>
   <parent link="table4_1"/>
   <child link="motor5_1"/>
-</joint>
+</joint> -->
 <joint name="motor6_joint" type="fixed">
   <origin xyz="-0.066956 -0.086535 0.0005" rpy="0 0 0"/>

Commit message: updated launch files

File: robot_arm_description/urdf/robot_arm.xacro (robot description, xacro)
@@ -524,5 +524,5 @@
   <child link="table1_1"/>
   <axis xyz="0.0 0.0 1.0"/>
-  <limit upper="1.570796" lower="-1.570796" effort="100" velocity="100"/>
+  <limit upper="1.57" lower="-1.57" effort="100" velocity="100"/>
 </joint>
 <joint name="tbone_joint" type="revolute">
@@ -557,5 +557,5 @@
   <child link="table5_1"/>
   <axis xyz="1.0 0.000515 0.0"/>
-  <limit upper="0.0" lower="-3.141593" effort="100" velocity="100"/>
+  <limit upper="1.57" lower="-1.57" effort="100" velocity="100"/>
 </joint>
 <joint name="motor1_joint" type="fixed">
