Commit message: Add files via upload

File: arm_description/urdf/arm.xacro (robot description, xacro)
@@ -4,9 +4,10 @@
 <xacro:include filename="$(find arm_description)/urdf/arm.trans" />
 <xacro:include filename="$(find arm_description)/urdf/arm.gazebo" />
+<xacro:include filename="ros2_control.xacro" />
 <link name="base_link">
   <inertial>
-    <origin xyz="-4.624614403843058e-14 -1.194549846011122e-16 0.0275289472946314" rpy="0 0 0"/>
-    <mass value="8.36745892677585"/>
-    <inertia ixx="0.018718" iyy="0.018718" izz="0.029518" ixy="-0.0" iyz="-0.0" ixz="-0.0"/>
+    <origin xyz="2.6758679619289235e-14 0.0 0.02266233904051618" rpy="0 0 0"/>
+    <mass value="2.5346787978702183"/>
+    <inertia ixx="0.005207" iyy="0.005207" izz="0.009019" ixy="-0.0" iyz="-0.0" ixz="0.0"/>
   </inertial>
   <visual>
@@ -15,5 +16,5 @@
       <mesh filename="file://$(find arm_description)/meshes/base_link.stl" scale="0.001 0.001 0.001"/>
     </geometry>
-    <material name="silver"/>
+    <material name="blue"/>
   </visual>
   <collision>
@@ -24,27 +25,7 @@
   </collision>
 </link>
-<link name="pipe_a_v3_1">
-  <inertial>
-    <origin xyz="-3.750134727944099e-08 0.004307791691554187 0.09000000000000004" rpy="0 0 0"/>
-    <mass value="0.09459182309374506"/>
-    <inertia ixx="0.000276" iyy="0.000272" izz="3.7e-05" ixy="0.0" iyz="-0.0" ixz="0.0"/>
-  </inertial>
-  <visual>
-    <origin xyz="-0.0 -0.0 -0.0" rpy="0 0 0"/>
-    <geometry>
-      <mesh filename="file://$(find arm_description)/meshes/pipe_a_v3_1.stl" scale="0.001 0.001 0.001"/>
-    </geometry>
-    <material name="silver"/>
-  </visual>
-  <collision>
-    <origin xyz="-0.0 -0.0 -0.0" rpy="0 0 0"/>
-    <geometry>
-      <mesh filename="file://$(find arm_description)/meshes/pipe_a_v3_1.stl" scale="0.001 0.001 0.001"/>
-    </geometry>
-  </collision>
-</link>
 <link name="pulley_c_v9_1">
   <inertial>
-    <origin xyz="-3.711542334716402e-17 3.465418341771916e-17 0.017705669740652963" rpy="0 0 0"/>
+    <origin xyz="-5.567313502074602e-17 4.098862764811248e-17 -0.003294330259347028" rpy="0 0 0"/>
     <mass value="0.05283781710784995"/>
     <inertia ixx="2.4e-05" iyy="2.4e-05" izz="3.8e-05" ixy="-0.0" iyz="0.0" ixz="-0.0"/>
@@ -55,5 +36,5 @@
       <mesh filename="file://$(find arm_description)/meshes/pulley_c_v9_1.stl" scale="0.001 0.001 0.001"/>
     </geometry>
-    <material name="silver"/>
+    <material name="iron"/>
   </visual>
   <collision>
@@ -66,19 +47,839 @@
 <link name="shoulder_bearling_house_prt1_v14_1">
   <inertial>
-    <origin xyz="4.208209917266138e-06 2.4287672296821914e-06 0.0040998460138022275" rpy="0 0 0"/>
+    <origin xyz="4.208209917286061e-06 2.4287672297167474e-06 -0.012900153986197746" rpy="0 0 0"/>
+    <mass value="0.057783249767342296"/>
+    <inertia ixx="3.6e-05" iyy="3.6e-05" izz="7.1e-05" ixy="-0.0" iyz="0.0" ixz="0.0"/>
+  </inertial>
+  <visual>
+    <origin xyz="-0.0 -0.0 -0.123" rpy="0 0 0"/>
+    <geometry>
+      <mesh filename="file://$(find arm_description)/meshes/shoulder_bearling_house_prt1_v14_1.stl" scale="0.001 0.001 0.001"/>
+    </geometry>
+    <material name="blue"/>
+  </visual>
+  <collision>
+    <origin xyz="-0.0 -0.0 -0.123" rpy="0 0 0"/>
+    <geometry>
+      <mesh filename="file://$(find arm_description)/meshes/shoulder_bearling_house_prt1_v14_1.stl" scale="0.001 0.001 0.001"/>
+    </geometry>
+  </collision>
+</link>
+<link name="table1_v2_1">
+  <inertial>
+    <origin xyz="-0.01893394777000812 -0.0198227756761575 0.008078541713728321" rpy="0 0 0"/>
+    <mass value="0.9953039551471342"/>
+    <inertia ixx="0.002494" iyy="0.002414" izz="0.004866" ixy="-9.6e-05" iyz="2e-06" ixz="-1e-06"/>
+  </inertial>
+  <visual>
+    <origin xyz="-0.0 -0.0 -0.1344" rpy="0 0 0"/>
+    <geometry>
+      <mesh filename="file://$(find arm_description)/meshes/table1_v2_1.stl" scale="0.001 0.001 0.001"/>
+    </geometry>
+    <material name="blue"/>
+  </visual>
+  <collision>
+    <origin xyz="-0.0 -0.0 -0.1344" rpy="0 0 0"/>
+    <geometry>
+      <mesh filename="file://$(find arm_description)/meshes/table1_v2_1.stl" scale="0.001 0.001 0.001"/>
+    </geometry>
+  </collision>
+</link>
+<link name="shoulder_bearling_house_prt3_v2_1">
+  <inertial>
+    <origin xyz="-3.326885494954389e-06 -9.453818210990768e-11 0.004385481296303423" rpy="0 0 0"/>
+    <mass value="0.05938208856291772"/>
+    <inertia ixx="3.7e-05" iyy="3.7e-05" izz="7.3e-05" ixy="0.0" iyz="-0.0" ixz="-0.0"/>
+  </inertial>
+  <visual>
+    <origin xyz="-0.0 -0.0 -0.1504" rpy="0 0 0"/>
+    <geometry>
+      <mesh filename="file://$(find arm_description)/meshes/shoulder_bearling_house_prt3_v2_1.stl" scale="0.001 0.001 0.001"/>
+    </geometry>
+    <material name="blue"/>
+  </visual>
+  <collision>
+    <origin xyz="-0.0 -0.0 -0.1504" rpy="0 0 0"/>
+    <geometry>
+      <mesh filename="file://$(find arm_description)/meshes/shoulder_bearling_house_prt3_v2_1.stl" scale="0.001 0.001 0.001"/>
+    </geometry>
+  </collision>
+</link>
+<link name="shoulder_v2_1">
+  <inertial>
+    <origin xyz="-0.05003301392386567 0.00744711420020433 0.06537453945113983" rpy="0 0 0"/>
+    <mass value="0.7582173734794716"/>
+    <inertia ixx="0.001635" iyy="0.002653" izz="0.001251" ixy="0.0" iyz="0.000136" ixz="-1e-06"/>
+  </inertial>
+  <visual>
+    <origin xyz="-0.05 0.095 -0.1504" rpy="0 0 0"/>
+    <geometry>
+      <mesh filename="file://$(find arm_description)/meshes/shoulder_v2_1.stl" scale="0.001 0.001 0.001"/>
+    </geometry>
+    <material name="blue"/>
+  </visual>
+  <collision>
+    <origin xyz="-0.05 0.095 -0.1504" rpy="0 0 0"/>
+    <geometry>
+      <mesh filename="file://$(find arm_description)/meshes/shoulder_v2_1.stl" scale="0.001 0.001 0.001"/>
+    </geometry>
+  </collision>
+</link>
+<link name="plangearbox1_v2_1">
+  <inertial>
+    <origin xyz="-2.198402479996289e-05 0.04289853923367516 7.979625855469852e-06" rpy="0 0 0"/>
+    <mass value="2.0006291062763104"/>
+    <inertia ixx="0.001765" iyy="0.000982" izz="0.001764" ixy="0.0" iyz="1e-06" ixz="-0.0"/>
+  </inertial>
+  <visual>
+    <origin xyz="2.4e-05 0.097184 -0.1954" rpy="0 0 0"/>
+    <geometry>
+      <mesh filename="file://$(find arm_description)/meshes/plangearbox1_v2_1.stl" scale="0.001 0.001 0.001"/>
+    </geometry>
+    <material name="black"/>
+  </visual>
+  <collision>
+    <origin xyz="2.4e-05 0.097184 -0.1954" rpy="0 0 0"/>
+    <geometry>
+      <mesh filename="file://$(find arm_description)/meshes/plangearbox1_v2_1.stl" scale="0.001 0.001 0.001"/>
+    </geometry>
+  </collision>
+</link>
+<link name="stepper1_v2_1">
+  <inertial>
+    <origin xyz="-2.2452245726494987e-05 0.04805206213786515 3.443202523836786e-05" rpy="0 0 0"/>
+    <mass value="0.47672097000804026"/>
+    <inertia ixx="0.000488" iyy="0.000235" izz="0.000488" ixy="0.0" iyz="-1e-06" ixz="-0.0"/>
+  </inertial>
+  <visual>
+    <origin xyz="6.7e-05 0.013684 -0.1954" rpy="0 0 0"/>
+    <geometry>
+      <mesh filename="file://$(find arm_description)/meshes/stepper1_v2_1.stl" scale="0.001 0.001 0.001"/>
+    </geometry>
+    <material name="black"/>
+  </visual>
+  <collision>
+    <origin xyz="6.7e-05 0.013684 -0.1954" rpy="0 0 0"/>
+    <geometry>
+      <mesh filename="file://$(find arm_description)/meshes/stepper1_v2_1.stl" scale="0.001 0.001 0.001"/>
+    </geometry>
+  </collision>
+</link>
+<link name="shoulder_bearling_house2_prt3_v3_1">
+  <inertial>
+    <origin xyz="-4.0536114861531317e-07 -0.0059858275962992105 -9.453793303748625e-11" rpy="0 0 0"/>
+    <mass value="0.05938208856291783"/>
+    <inertia ixx="3.7e-05" iyy="7.3e-05" izz="3.7e-05" ixy="-0.0" iyz="0.0" ixz="0.0"/>
+  </inertial>
+  <visual>
+    <origin xyz="4.5e-05 0.055884 -0.2754" rpy="0 0 0"/>
+    <geometry>
+      <mesh filename="file://$(find arm_description)/meshes/shoulder_bearling_house2_prt3_v3_1.stl" scale="0.001 0.001 0.001"/>
+    </geometry>
+    <material name="blue"/>
+  </visual>
+  <collision>
+    <origin xyz="4.5e-05 0.055884 -0.2754" rpy="0 0 0"/>
+    <geometry>
+      <mesh filename="file://$(find arm_description)/meshes/shoulder_bearling_house2_prt3_v3_1.stl" scale="0.001 0.001 0.001"/>
+    </geometry>
+  </collision>
+</link>
+<link name="new_pipe_b_v8_1">
+  <inertial>
+    <origin xyz="-3.1295264940206456e-05 0.05999962743199911 0.002489679948011303" rpy="0 0 0"/>
+    <mass value="0.08655426473406591"/>
+    <inertia ixx="0.000229" iyy="3.8e-05" izz="0.000226" ixy="0.0" iyz="-0.0" ixz="-0.0"/>
+  </inertial>
+  <visual>
+    <origin xyz="2.1e-05 0.102029 -0.2754" rpy="0 0 0"/>
+    <geometry>
+      <mesh filename="file://$(find arm_description)/meshes/new_pipe_b_v8_1.stl" scale="0.001 0.001 0.001"/>
+    </geometry>
+    <material name="black"/>
+  </visual>
+  <collision>
+    <origin xyz="2.1e-05 0.102029 -0.2754" rpy="0 0 0"/>
+    <geometry>
+      <mesh filename="file://$(find arm_description)/meshes/new_pipe_b_v8_1.stl" scale="0.001 0.001 0.001"/>
+    </geometry>
+  </collision>
+</link>
+<link name="shoulder_bearling_house_2prt1_v5_1">
+  <inertial>
+    <origin xyz="4.24595728622469e-06 -0.004300516777600696 -4.207479079365584e-06" rpy="0 0 0"/>
     <mass value="0.05778324976734234"/>
-    <inertia ixx="3.6e-05" iyy="3.6e-05" izz="7.1e-05" ixy="-0.0" iyz="0.0" ixz="0.0"/>
-  </inertial>
-  <visual>
-    <origin xyz="-0.0 0.0 -0.123" rpy="0 0 0"/>
-    <geometry>
-      <mesh filename="file://$(find arm_description)/meshes/shoulder_bearling_house_prt1_v14_1.stl" scale="0.001 0.001 0.001"/>
-    </geometry>
-    <material name="silver"/>
-  </visual>
-  <collision>
-    <origin xyz="-0.0 0.0 -0.123" rpy="0 0 0"/>
-    <geometry>
-      <mesh filename="file://$(find arm_description)/meshes/shoulder_bearling_house_prt1_v14_1.stl" scale="0.001 0.001 0.001"/>
+    <inertia ixx="3.6e-05" iyy="7.1e-05" izz="3.6e-05" ixy="-0.0" iyz="-0.0" ixz="0.0"/>
+  </inertial>
+  <visual>
+    <origin xyz="2.1e-05 0.102029 -0.2754" rpy="0 0 0"/>
+    <geometry>
+      <mesh filename="file://$(find arm_description)/meshes/shoulder_bearling_house_2prt1_v5_1.stl" scale="0.001 0.001 0.001"/>
+    </geometry>
+    <material name="blue"/>
+  </visual>
+  <collision>
+    <origin xyz="2.1e-05 0.102029 -0.2754" rpy="0 0 0"/>
+    <geometry>
+      <mesh filename="file://$(find arm_description)/meshes/shoulder_bearling_house_2prt1_v5_1.stl" scale="0.001 0.001 0.001"/>
+    </geometry>
+  </collision>
+</link>
+<link name="shoulder_bearling_house2_prt2_v10_1">
+  <inertial>
+    <origin xyz="-7.534969931434021e-06 0.00999965589472103 7.596384632435615e-11" rpy="0 0 0"/>
+    <mass value="0.17595730314710867"/>
+    <inertia ixx="0.000105" iyy="0.000198" izz="0.000105" ixy="-0.0" iyz="0.0" ixz="-0.0"/>
+  </inertial>
+  <visual>
+    <origin xyz="3e-05 0.085884 -0.2754" rpy="0 0 0"/>
+    <geometry>
+      <mesh filename="file://$(find arm_description)/meshes/shoulder_bearling_house2_prt2_v10_1.stl" scale="0.001 0.001 0.001"/>
+    </geometry>
+    <material name="blue"/>
+  </visual>
+  <collision>
+    <origin xyz="3e-05 0.085884 -0.2754" rpy="0 0 0"/>
+    <geometry>
+      <mesh filename="file://$(find arm_description)/meshes/shoulder_bearling_house2_prt2_v10_1.stl" scale="0.001 0.001 0.001"/>
+    </geometry>
+  </collision>
+</link>
+<link name="tbone_v1_1">
+  <inertial>
+    <origin xyz="-0.0001179461306405897 -0.040037043730441445 0.011561726312559306" rpy="0 0 0"/>
+    <mass value="0.7230946223073603"/>
+    <inertia ixx="0.000893" iyy="0.000815" izz="0.000779" ixy="0.0" iyz="-0.0" ixz="-1e-06"/>
+  </inertial>
+  <visual>
+    <origin xyz="9.6e-05 -0.042971 -0.2754" rpy="0 0 0"/>
+    <geometry>
+      <mesh filename="file://$(find arm_description)/meshes/tbone_v1_1.stl" scale="0.001 0.001 0.001"/>
+    </geometry>
+    <material name="blue"/>
+  </visual>
+  <collision>
+    <origin xyz="9.6e-05 -0.042971 -0.2754" rpy="0 0 0"/>
+    <geometry>
+      <mesh filename="file://$(find arm_description)/meshes/tbone_v1_1.stl" scale="0.001 0.001 0.001"/>
+    </geometry>
+  </collision>
+</link>
+<link name="pipe_c_v1_1">
+  <inertial>
+    <origin xyz="-0.00013201873724399225 0.004305319532101214 0.029999580087758992" rpy="0 0 0"/>
+    <mass value="0.03153060769791503"/>
+    <inertia ixx="1.6e-05" iyy="1.5e-05" izz="1.2e-05" ixy="0.0" iyz="0.0" ixz="0.0"/>
+  </inertial>
+  <visual>
+    <origin xyz="0.0002 -0.002971 -0.308202" rpy="0 0 0"/>
+    <geometry>
+      <mesh filename="file://$(find arm_description)/meshes/pipe_c_v1_1.stl" scale="0.001 0.001 0.001"/>
+    </geometry>
+    <material name="black"/>
+  </visual>
+  <collision>
+    <origin xyz="0.0002 -0.002971 -0.308202" rpy="0 0 0"/>
+    <geometry>
+      <mesh filename="file://$(find arm_description)/meshes/pipe_c_v1_1.stl" scale="0.001 0.001 0.001"/>
+    </geometry>
+  </collision>
+</link>
+<link name="table2_v1_1">
+  <inertial>
+    <origin xyz="-6.1229488199372305e-06 -0.01939156035360563 0.021075670529906776" rpy="0 0 0"/>
+    <mass value="0.4458483416017101"/>
+    <inertia ixx="0.000644" iyy="0.000372" izz="0.000968" ixy="1e-06" iyz="2.3e-05" ixz="0.0"/>
+  </inertial>
+  <visual>
+    <origin xyz="0.0002 -0.002971 -0.368202" rpy="0 0 0"/>
+    <geometry>
+      <mesh filename="file://$(find arm_description)/meshes/table2_v1_1.stl" scale="0.001 0.001 0.001"/>
+    </geometry>
+    <material name="blue"/>
+  </visual>
+  <collision>
+    <origin xyz="0.0002 -0.002971 -0.368202" rpy="0 0 0"/>
+    <geometry>
+      <mesh filename="file://$(find arm_description)/meshes/table2_v1_1.stl" scale="0.001 0.001 0.001"/>
+    </geometry>
+  </collision>
+</link>
+<link name="arm_plate_v2_1">
+  <inertial>
+    <origin xyz="-2.1378266405119113e-06 0.004999567309755676 0.12307397675626303" rpy="0 0 0"/>
+    <mass value="0.46224273474069966"/>
+    <inertia ixx="0.002956" iyy="0.003113" izz="0.000168" ixy="-0.0" iyz="-0.0" ixz="-0.0"/>
+  </inertial>
+  <visual>
+    <origin xyz="0.000157 0.081029 -0.398202" rpy="0 0 0"/>
+    <geometry>
+      <mesh filename="file://$(find arm_description)/meshes/arm_plate_v2_1.stl" scale="0.001 0.001 0.001"/>
+    </geometry>
+    <material name="blue"/>
+  </visual>
+  <collision>
+    <origin xyz="0.000157 0.081029 -0.398202" rpy="0 0 0"/>
+    <geometry>
+      <mesh filename="file://$(find arm_description)/meshes/arm_plate_v2_1.stl" scale="0.001 0.001 0.001"/>
+    </geometry>
+  </collision>
+</link>
+<link name="bearing_holder_elbow_v3_1">
+  <inertial>
+    <origin xyz="-6.845835323396126e-06 0.01201199759666062 0.0003832891577878472" rpy="0 0 0"/>
+    <mass value="0.2912306079023313"/>
+    <inertia ixx="0.000136" iyy="0.000186" izz="0.000138" ixy="-0.0" iyz="3e-06" ixz="-0.0"/>
+  </inertial>
+  <visual>
+    <origin xyz="0.000156 0.082029 -0.628362" rpy="0 0 0"/>
+    <geometry>
+      <mesh filename="file://$(find arm_description)/meshes/bearing_holder_elbow_v3_1.stl" scale="0.001 0.001 0.001"/>
+    </geometry>
+    <material name="blue"/>
+  </visual>
+  <collision>
+    <origin xyz="0.000156 0.082029 -0.628362" rpy="0 0 0"/>
+    <geometry>
+      <mesh filename="file://$(find arm_description)/meshes/bearing_holder_elbow_v3_1.stl" scale="0.001 0.001 0.001"/>
+    </geometry>
+  </collision>
+</link>
+<link name="elbow_joint_axes_v5_1">
+  <inertial>
+    <origin xyz="-1.6827600113223566e-05 0.03187463876334105 0.00016453920275805167" rpy="0 0 0"/>
+    <mass value="0.4827163962244698"/>
+    <inertia ixx="0.000198" iyy="0.000151" izz="0.000198" ixy="0.0" iyz="1e-06" ixz="-0.0"/>
+  </inertial>
+  <visual>
+    <origin xyz="0.000151 0.091029 -0.628362" rpy="0 0 0"/>
+    <geometry>
+      <mesh filename="file://$(find arm_description)/meshes/elbow_joint_axes_v5_1.stl" scale="0.001 0.001 0.001"/>
+    </geometry>
+    <material name="blue"/>
+  </visual>
+  <collision>
+    <origin xyz="0.000151 0.091029 -0.628362" rpy="0 0 0"/>
+    <geometry>
+      <mesh filename="file://$(find arm_description)/meshes/elbow_joint_axes_v5_1.stl" scale="0.001 0.001 0.001"/>
+    </geometry>
+  </collision>
+</link>
+<link name="elbow_side_plate_v3_1">
+  <inertial>
+    <origin xyz="0.016154358279447927 -0.0014598177767405976 -1.5816912823929385e-07" rpy="0 0 0"/>
+    <mass value="0.3773934236223084"/>
+    <inertia ixx="0.000159" iyy="0.000733" izz="0.000577" ixy="-0.0" iyz="0.0" ixz="-0.0"/>
+  </inertial>
+  <visual>
+    <origin xyz="0.000174 0.047929 -0.628362" rpy="0 0 0"/>
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
File: arm_description/urdf/materials.xacro (robot description, xacro)
@@ -4,3 +4,12 @@
   <color rgba="0.700 0.700 0.700 1.000"/>
 </material>
+<material name="black">
+  <color rgba="0.05 0.05 0.05 1.000"/>
+</material>
+<material name="blue">
+  <color rgba="0.015 0.015 0.700 1.000"/>
+</material>
+<material name="iron">
+  <color rgba="0.700 0.700 0.800 1.000"/>
+</material>
 </robot>
